File: hw/Zvuk9_R2.brd (EAGLE design)
At the start: 330.1 x 84.6 mm, 149 parts, among them Q1 FDC6312P, Q2 FDC6312P, SW1 B3F-3122, U1 4067-SO24W, U2 4067-SO24W, U3 4067-SO24W, U4 4067-SO24W, U5 AT90USB1286, U6 74HCT165, U7 74HCT238SO, U8 ULN2803ADW, U9 74HCT138SO, Y1 16MHz

Commit message: refactor the entire codebase, port to stm32
Parts:
- removed CONN6: PINHD-2X05-TH-2.54MM-V, igor_lbr:2X05-2.54-V
- removed CONN7: PINHD-1X03-TH-2.54MM, igor_lbr:1X03-2.54-V
- removed D26: BAW56, igor_lbr:SOT23
- removed D27, D28, D29, D30, D31, D32, D33, D34, D35, D36, D37, D38, D39, D40, D41, D42, D43, D44, D45, D46, D47, D48: White, igor_lbr:0805_LED
- removed R3: 10k, igor_lbr:R0603
- added C25, C26: 18p, igor_lbr:C0805
- added C27: 100n, igor_lbr:C0805
- C1: device igor_lbr:153CLV-0405 -> igor_lbr:C-TH-E-0502
- C10, C11, C12, C13, C14, C15, C17, C18, C19, C2, C20, C21, C22, C23, C24, C4, C5, C8, C9: device igor_lbr:C0603 -> igor_lbr:C0805
- C16: value 100n -> 1u; device igor_lbr:C0603 -> igor_lbr:C0805
- C3: value 1u -> 2.2u; device igor_lbr:C0603 -> igor_lbr:C0805
- C6: value 22p -> 2.2u; device igor_lbr:C0603 -> igor_lbr:C0805
- C7: value 22p -> 100n; device igor_lbr:C0603 -> igor_lbr:C0805
- CONN1: value USB-B-PTH -> USB-B-H
- CONN3: value PINHD-2X03-TH-2.54MM-V -> PINHD-1X03-TH-2.54MM; device igor_lbr:2X03-2.54-V -> igor_lbr:1X03-2.54-V
- CONN4, CONN5: device igor_lbr:FFC-18P-SMD-1MM-MOLEX-52271-1879 -> igor_lbr:MOLEX-52271-1879
- D7: value Orange -> BAW56; device igor_lbr:0805_LED -> igor_lbr:SOT23
- ENC10, ENC4, ENC5, ENC6, ENC7, ENC8, ENC9: value ALPS-EC12E24204A7 -> ALPS-EC12E24404AX; device igor_lbr:ALPS-EC12-STD-17.5MM -> igor_lbr:EC12E-1
- ENC2: value ALPS-EC12E24204A7 -> ALPS-EC12D1524403; device igor_lbr:ALPS-EC12-STD-17.5MM -> igor_lbr:ALPS_EC12-SW
- ENC3: value ALPS-EC12D1524403 -> ALPS-EC12E24404AX; device igor_lbr:ALPS_EC12-SW -> igor_lbr:EC12E-1
- R1: value 10k -> 510; device igor_lbr:R0603 -> igor_lbr:R0805
- R10, R12, R8: value 4k7 -> 4.7k; device igor_lbr:R0603 -> igor_lbr:R0805
- R11, R13, R9: value 36 -> 22; device igor_lbr:R0603 -> igor_lbr:R0805
- R14, R15, R16, R17, R18, R19, R20, R21: value 10k -> 4.7k; device igor_lbr:R0603 -> igor_lbr:R0805
- R2: value 1k -> 4.7k; device igor_lbr:R0603 -> igor_lbr:R0805
- R4, R5: device igor_lbr:R0603 -> igor_lbr:R0805
- R6: value 220 -> 10; device igor_lbr:R0603 -> igor_lbr:R0805
- R7: value 220 -> 33; device igor_lbr:R0603 -> igor_lbr:R0805
- SW1: value B3F-3122 -> OMRON-B3W-9; device igor_lbr:B3F-312X -> igor_lbr:OMRON-B3W-9
- SW10, SW11, SW12, SW13, SW14, SW15, SW16, SW17, SW18, SW19, SW2, SW20, SW21, SW22, SW3, SW4, SW5, SW6, SW7, SW8, SW9: value (none) -> OMRON-B3W-9; device igor_lbr:RUBBER_SWITCH -> igor_lbr:OMRON-B3W-9
- SW23: device igor_lbr:RUBBER_SWITCH -> igor_lbr:B3F-312X
- U1, U2, U3, U4: value 4067-SO24W -> MC14067BDWR2G-SO24W
- U5: value AT90USB1286 -> STM32F405RGT6-10X10-HS; device igor_lbr:TQFP-64-14X14 -> igor_lbr:TQFP-64-10X10-HS
- U6: value 74HCT165 -> 74HC165
- U7: value 74HCT238SO -> 74238-SO
- U8: value ULN2803ADW -> ULN2803A-SO
- U9: value 74HCT138SO -> 74138-SO
- VR2: value MCP1825 -> AP7343-SOT25; device igor_lbr:SOT223 -> igor_lbr:SOT25
- moved ENC2 306.9 mm to (13.2, 33.4)
- moved D23 285.3 mm to (20.6, 43.2), turned to 0 degrees
- moved D20 279.8 mm to (15.9, 43.2), turned to 0 degrees
- moved D13 268.4 mm to (10.9, 63.5), turned to 0 degrees
- moved D5 258.2 mm to (6.48, 63.5)
- moved D9 254.6 mm to (6.48, 43.2)
- moved ENC3 245.2 mm to (258.4, 53.7)
- moved D17 243.8 mm to (11.2, 43.2)
- moved D12 198.6 mm to (221.6, 23.2)
- moved D2 187.2 mm to (73.3, 23.2)
- moved D4 175.0 mm to (214.0, 57.9), turned to 0 degrees
- moved SW8 144.9 mm to (232.2, 51.1)
- moved D10 121.6 mm to (161.5, 23.2), turned to 0 degrees
- moved SW23 120.8 mm to (48.0, 81.5), flipped to the bottom, turned to 180 degrees
- moved D6 110.7 mm to (161.5, 42.9), turned to 0 degrees
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Connections:
- net N$12 renamed USB_SHIELD
- removed net AREF: C19.1, CONN7.1, VR2.3
- removed net AREF_SELECT: C11.1, C12.1, C4.1, C5.1, CONN7.2, U1.24, U2.24, U3.24, U4.24, U5.62
- removed net BTLDR_EN: R3.2, SW1.1, U5.43
- removed net IN_COLUMN_0: ENC1.C, ENC3.C, ENC5.C, ENC7.C, U9.15
- removed net IN_COLUMN_1: ENC2.C, ENC4.C, ENC6.C, ENC9.C, U9.14
- removed net IN_COLUMN_2: ENC10.C, ENC8.C, U9.13
- removed net IN_COLUMN_3: SW10.1, SW14.1, SW17.1, SW19.1, SW21.1, SW22.1, SW4.1, SW8.1, U9.12
- removed net IN_COLUMN_4: SW12.1, SW15.1, SW16.1, SW18.1, SW2.1, SW20.1, SW23.1, SW6.1, U9.11
- removed net IN_COLUMN_5: ENC1.D, SW13.1, SW5.1, SW9.1, U9.10
- removed net IN_COLUMN_6: ENC3.D, SW11.1, SW3.1, SW7.1, U9.9
- removed net IN_COLUMN_7: U9.7
- removed net IN_ROW_0: D11.3, D12.3, D13.3, D26.3, R17.1, U6.11
- removed net IN_ROW_1: D10.3, D2.3, D25.3, D8.3, R16.1, U6.12
- removed net IN_ROW_2: D24.3, D4.3, D5.3, D6.3, R15.1, U6.13
- removed net IN_ROW_3: D1.3, D23.3, D3.3, D9.3, R14.1, U6.14
- removed net IN_ROW_4: D16.3, D21.3, R18.1, U6.3
- removed net IN_ROW_5: D18.3, D19.3, R19.1, U6.4
- removed net IN_ROW_6: D17.3, D20.3, R20.1, U6.5
- removed net IN_ROW_7: D15.3, D22.3, R21.1, U6.6
- removed net LR_1_L: D27.A, D30.A, D33.A, D36.A, D39.A, D42.A, D45.A, D48.A, R9.2
- removed net LR_1_Q: Q1.1, R8.2, U5.15
- removed net LR_2_L: D28.A, D31.A, D34.A, D37.A, D40.A, D43.A, D46.A, R11.2
- removed net LR_2_Q: Q1.3, R10.2, U5.16
- removed net LR_3_L: D29.A, D32.A, D35.A, D38.A, D41.A, D44.A, D47.A, R13.2
- removed net LR_3_Q: Q2.3, R12.2, U5.14
- removed net MISO: CONN3.1, U5.13
- removed net MUX_COMMON_0/TDI: CONN6.9, U1.1, U5.54
- removed net MUX_COMMON_1/TMS: CONN6.5, U2.1, U5.56
- removed net MUX_COMMON_2/TDO: CONN6.3, U3.1, U5.55
- removed net MUX_COMMON_3/TCK: CONN6.1, U4.1, U5.57
- removed net N$32: D5.2, SW9.2
- removed net N$33: D5.1, SW7.2
- removed net N$34: D9.2, SW13.2
- removed net N$35: D9.1, SW11.2
- removed net N$36: D12.2, ENC1.E
- removed net N$40: D12.1, ENC3.E
- removed net RESET: CONN3.5, CONN6.6, R1.2, U5.20
- removed net SDA: U5.26
- removed net SR_CLOCK: U5.31, U6.2
- removed net SR_LATCH: U5.32, U6.1
- removed net SR_OUT: U5.30, U6.9
- removed net TX: R6.2, U5.28
- removed net UCAP: C3.2, U5.7
- removed net XTAL1: C6.1, U5.24, Y1.1
- removed net XTAL2: C7.1, U5.23, Y1.2
- new net +3V3: C10.1, C11.1, C12.1, C13.1, C15.1, C16.1, C19.1, C20.2, C21.2, C22.2, C23.1, C24.1, C4.1, C5.1, C7.1, C8.1, R14.2, R15.2, R16.2, R17.2, R18.2, R19.2, R20.2, R21.2, R7.2, U1.24, U2.24, U3.24, U4.24, U5.1, U5.13, U5.19, U5.32, U5.48, U5.64, U6.16, U7.16, U7.6, U8.10, U9.16, U9.6, VR2.5
- new net BC1: ENC1.C, ENC1.D, ENC2.C, ENC2.D, SW1.1, U9.15
- new net BC2: ENC3.C, ENC7.C, SW16.1, SW3.1, SW9.1, U9.14
- new net BC3: ENC4.C, ENC8.C, SW10.1, SW17.1, SW2.1, U9.13
- new net BC4: ENC5.C, ENC9.C, SW11.1, SW18.1, SW4.1, U9.12
- new net BC5: ENC10.C, ENC6.C, SW12.1, SW19.1, SW5.1, U9.11
- new net BC6: SW13.1, SW20.1, SW6.1, U9.10
- new net BC7: SW14.1, SW21.1, SW7.1, U9.9
- new net BC8: SW15.1, SW22.1, SW8.1, U9.7
- new net BOOT0: R1.1, U5.60
- new net BR1: D1.3, D2.3, D3.3, D4.3, R14.1, U6.11
- new net BR2: D5.3, D6.3, D7.3, D8.3, R15.1, U6.12
- new net BR3: D10.3, D11.3, D12.3, D9.3, R16.1, U6.13
- new net BR4: R17.1, U6.14
- new net BR5: D13.3, D15.3, D16.3, R18.1, U6.3
- new net BR6: D17.3, D18.3, D19.3, R19.1, U6.4
- new net BR7: D20.3, D21.3, D22.3, R20.1, U6.5
- new net BR8: D23.3, D24.3, D25.3, R21.1, U6.6
- new net BTLDR_BUTTON: R2.1, SW23.1, U5.24
- new net LR_1_MI: Q1.1, R8.2, U5.57
- new net LR_1_MO: R9.2, SW1.6-A, SW2.6-A, SW3.6-A, SW4.6-A, SW5.6-A, SW6.6-A, SW7.6-A, SW8.6-A
- new net LR_2_MI: Q1.3, R10.2, U5.56
- new net LR_2_MO: R11.2, SW10.6-A, SW11.6-A, SW12.6-A, SW13.6-A, SW14.6-A, SW15.6-A, SW9.6-A
- new net LR_3_MI: Q2.3, R12.2, U5.55
- new net LR_3_MO: R13.2, SW16.6-A, SW17.6-A, SW18.6-A, SW19.6-A, SW20.6-A, SW21.6-A, SW22.6-A
- new net MIDI_OUT: R6.2, U5.29
- new net MUX_COMMON_1: U1.1, U5.17
- new net MUX_COMMON_2: U2.1, U5.14
- new net MUX_COMMON_3: U3.1, U5.15
- new net MUX_COMMON_4: U4.1, U5.16
- new net N$10: D3.2, SW5.3
- new net N$11: D3.1, SW6.3
- new net N$12: C3.2, U5.31
- new net N$13: C6.1, U5.47
- new net N$5: D1.1, SW1.3
- new net N$8: D2.1, SW4.3
- new net N$9: D1.2, SW3.3
- new net NRST: C27.1, U5.7
- new net OSC_IN: C25.1, U5.5, Y1.1
- new net OSC_OUT: C26.1, U5.6, Y1.2
- new net SR_IN_CLOCK: U5.4, U6.2
- new net SR_IN_DATA: U5.3, U6.9
- new net SR_IN_LATCH: U5.2, U6.1
- new net SWDCLK: CONN3.1, U5.49
- new net SWDIO: CONN3.2, U5.46
- net +5V: now also R2.2, VR2.3; no longer C10.1, C13.1, C15.1, C16.1, C20.2, C21.2, C22.2, C23.1, C24.1, C8.1, CONN3.2, CONN6.4, CONN7.3, R1.1, R14.2, R15.2, R16.2, R17.2, R18.2, R19.2, R2.1, R20.2, R21.2, R3.1, R7.2, U5.21, U5.3, U5.52, U5.64, U5.8, U6.16, U7.16, U7.6, U8.10, U9.16, U9.6
- net D+: now also U5.45; no longer U5.5
- net D-: now also U5.44; no longer U5.4
- net DEC_IN_A0: now also U5.39; no longer U5.38
- net DEC_IN_A1: now also U5.38; no longer U5.39
- net DEC_IN_A2: now also U5.37; no longer U5.40
- net DEC_OUT_A0: now also U5.62; no longer U5.35
- net DEC_OUT_A1: now also U5.59; no longer U5.36
- net DEC_OUT_A2: now also U5.58; no longer U5.37
- net E10_A: now also D22.1; no longer D25.1
- net E10_B: now also D25.1; no longer D26.1
- net E1_A: now also D13.1; no longer D3.1
- net E1_B: now also D17.1; no longer D6.1
- net E2_A: now also D20.1, ENC2.A; no longer D10.1, ENC3.A
- net E2_B: now also D23.1, ENC2.B; no longer D13.1, ENC3.B
- net E3_A: now also D13.2, ENC3.A; no longer D16.1, ENC5.A
- net E3_B: now also D17.2, ENC3.B; no longer D18.1, ENC5.B
- net E4_A: now also D15.1, ENC4.A; no longer D20.1, ENC7.A
- net E4_B: now also D18.1, ENC4.B; no longer D22.1, ENC7.B
- net E5_A: now also D15.2, ENC5.A; no longer D3.2, ENC9.A
- net E5_B: now also D18.2, ENC5.B; no longer D6.2, ENC9.B
- net E6_A: now also D16.1, ENC6.A; no longer D10.2, ENC2.A
- net E6_B: now also D19.1, ENC6.B; no longer D13.2, ENC2.B
- net E7_A: now also D20.2, ENC7.A; no longer D16.2, ENC4.A
- net E7_B: now also D23.2, ENC7.B; no longer D18.2, ENC4.B
- net E8_A: now also D21.1, ENC8.A; no longer D20.2, ENC6.A
- net E8_B: now also D24.1, ENC8.B; no longer D22.2, ENC6.B
- net E9_A: now also D21.2, ENC9.A; no longer D23.1, ENC8.A
- net E9_B: now also D24.2, ENC9.B; no longer D24.1, ENC8.B
- net GND: now also C25.2, C26.2, C27.2, CONN3.3, R1.2, SW23.2, U5.12, U5.18; no longer CONN3.6, CONN6.10, CONN6.2, D7.C, SW1.2, U5.22, U5.53, U5.6, VR2.4
- net LCD_CS: now also U5.52; no longer U5.47
- net LCD_DC: now also U5.54; no longer U5.48
- net LCD_RESET: now also U5.50; no longer U5.46
- net LC_1: now also SW15.6-C, SW22.6-C, SW8.6-C; no longer D27.C, D28.C, D29.C
- net LC_2: now also SW14.6-C, SW21.6-C, SW7.6-C; no longer D30.C, D31.C, D32.C
- net LC_3: now also SW13.6-C, SW20.6-C, SW6.6-C; no longer D33.C, D34.C, D35.C
- net LC_4: now also SW12.6-C, SW19.6-C, SW5.6-C; no longer D36.C, D37.C, D38.C
- net LC_5: now also SW11.6-C, SW18.6-C, SW4.6-C; no longer D39.C, D40.C, D41.C
- net LC_6: now also SW10.6-C, SW17.6-C, SW3.6-C; no longer D42.C, D43.C, D44.C
- net LC_7: now also SW16.6-C, SW2.6-C, SW9.6-C; no longer D45.C, D46.C, D47.C
- net LC_8: now also SW1.6-C; no longer D48.C
- net MOSI: now also U5.53; no longer CONN3.4, U5.12
- net MUX_S0: now also U5.33; no longer U5.60
- net MUX_S1: now also U5.34; no longer U5.61
- net MUX_S2: now also U5.36; no longer U5.59
- net MUX_S3: now also U5.35; no longer U5.58
- net N$14: now also D4.2, SW7.3; no longer D1.2, SW4.2
- net N$15: now also D4.1, SW8.3; no longer D1.1, SW2.2
- net N$16: now also D5.2, ENC1.E; no longer D4.2, SW8.2
- net N$17: now also D6.2, SW10.3; no longer D4.1, SW6.2
- net N$18: now also D6.1, SW11.3; no longer D8.1, SW10.2
- net N$19: now also D7.1, SW12.3; no longer D8.2, SW12.2
- net N$20: now also D7.2, SW13.3; no longer D11.1, SW14.2
- net N$21: now also D8.2, SW14.3; no longer D11.2, SW15.2
- net N$22: now also D8.1, SW15.3; no longer D15.2, SW17.2
- net N$23: now also D5.1, SW9.3; no longer D15.1, SW16.2
- net N$24: now also D9.2, ENC2.E; no longer D17.2, SW19.2
- net N$25: now also D9.1, SW16.3; no longer D17.1, SW18.2
- net N$26: now also D10.2, SW17.3; no longer D19.2, SW21.2
- net N$27: now also D10.1, SW18.3; no longer D19.1, SW20.2
- net N$28: now also D11.2, SW19.3; no longer D21.1, SW22.2
- net N$29: now also D11.1, SW20.3; no longer D21.2, SW23.2
- net N$30: now also D12.2, SW21.3; no longer D2.2, SW5.2
- net N$31: now also D12.1, SW22.3; no longer D2.1, SW3.2
- net N$6: now also D2.2, SW2.3; no longer D7.A, R2.2
- net SCLK: now also U5.51; no longer CONN3.3, U5.11
Routing:
- net BR7: track 0.00 -> 608.7 mm, vias 0 -> 4
- net BR8: track 0.00 -> 592.6 mm, vias 0 -> 8
- net BR6: track 0.00 -> 587.8 mm, vias 0 -> 6
- net +5V: track 786.5 -> 207.9 mm, vias 0 -> 2
- net IN_ROW_0: track 525.6 -> 0.00 mm, vias 5 -> 0
- net BR5: track 0.00 -> 515.0 mm, vias 0 -> 2
- net BC1: track 0.00 -> 427.1 mm, vias 0 -> 1
- net IN_ROW_3: track 412.6 -> 0.00 mm, vias 7 -> 0
- net E7_A: track 83.5 -> 492.2 mm, vias 2 -> 1
- net +3V3: track 0.00 -> 401.9 mm, vias 0 -> 1
- net BR2: track 0.00 -> 400.2 mm, vias 0 -> 9
- net IN_ROW_2: track 397.6 -> 0.00 mm, vias 4 -> 0
- net BR3: track 0.00 -> 374.9 mm, vias 0 -> 12
- net IN_COLUMN_4: track 365.0 -> 0.00 mm, vias 9 -> 0
- net LR_1_L: track 360.3 -> 0.00 mm, vias 22 -> 0
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Other:
- board size 330.1 x 84.6 mm -> 330.1 x 89 mm
- board text added: "GND"
- board text added: "SWDCLK"
- board text added: "SWDIO"
- board text added: "ZVUK9 R3 2021.06"
- board text removed: "3V3"
- board text removed: "5V"
- board text removed: "AREF SELECT"
- board text removed: "I.P."
- board text removed: "ICSP"
- board text removed: "JTAG"
- board text removed: "ZVUK9 R2 2016.12"
