File: hw/Zvuk9_R2.sch (EAGLE design)
At the start: 149 parts, among them Q1 FDC6312P, Q2 FDC6312P, SW1 B3F-3122, U1 4067-SO24W, U2 4067-SO24W, U3 4067-SO24W, U4 4067-SO24W, U5 AT90USB1286, U6 74HCT165, U7 74HCT238SO, U8 ULN2803ADW, U9 74HCT138SO, Y1 16MHz

Commit message: refactor the entire codebase, port to stm32
Parts:
- removed CONN6: PINHD-2X05-TH-2.54MM-V, igor_lbr:PINHD-2X05-TH-2.54MM-V
- removed CONN7: PINHD-1X03-TH-2.54MM, igor_lbr:PINHD-1X03-TH-2.54MM
- removed D26: BAW56, igor_lbr:BAW56
- removed D27, D28, D29, D30, D31, D32, D33, D34, D35, D36, D37, D38, D39, D40, D41, D42, D43, D44, D45, D46, D47, D48: White, igor_lbr:LED-0805
- removed R3: 10k, igor_lbr:RESISTOR-0603
- added C25, C26: 18p, igor_lbr:CAPACITOR-0805
- added C27: 100n, igor_lbr:CAPACITOR-0805
- C1: device igor_lbr:ELECTROLYTIC_CAPACITOR-CLV-0405 -> igor_lbr:ELECTROLYTIC_CAPACITOR-C-TH-E-0502
- C10, C11, C12, C13, C14, C15, C17, C18, C19, C2, C20, C21, C22, C23, C24, C4, C5, C8, C9: device igor_lbr:CAPACITOR-0603 -> igor_lbr:CAPACITOR-0805
- C16: value 100n -> 1u; device igor_lbr:CAPACITOR-0603 -> igor_lbr:CAPACITOR-0805
- C3: value 1u -> 2.2u; device igor_lbr:CAPACITOR-0603 -> igor_lbr:CAPACITOR-0805
- C6: value 22p -> 2.2u; device igor_lbr:CAPACITOR-0603 -> igor_lbr:CAPACITOR-0805
- C7: value 22p -> 100n; device igor_lbr:CAPACITOR-0603 -> igor_lbr:CAPACITOR-0805
- CONN1: value USB-B-PTH -> USB-B-H; device igor_lbr:USB-B-PTH -> igor_lbr:USB-B-H
- CONN3: value PINHD-2X03-TH-2.54MM-V -> PINHD-1X03-TH-2.54MM; device igor_lbr:PINHD-2X03-TH-2.54MM-V -> igor_lbr:PINHD-1X03-TH-2.54MM
- D7: value Orange -> BAW56; device igor_lbr:LED-0805 -> igor_lbr:BAW56
- ENC10, ENC4, ENC5, ENC6, ENC7, ENC8, ENC9: value ALPS-EC12E24204A7 -> ALPS-EC12E24404AX; device igor_lbr:ALPS-EC12E24204A7 -> igor_lbr:ALPS-EC12E24404AX
- ENC2: value ALPS-EC12E24204A7 -> ALPS-EC12D1524403; device igor_lbr:ALPS-EC12E24204A7 -> igor_lbr:ALPS-EC12D1524403
- ENC3: value ALPS-EC12D1524403 -> ALPS-EC12E24404AX; device igor_lbr:ALPS-EC12D1524403 -> igor_lbr:ALPS-EC12E24404AX
- R1: value 10k -> 510; device igor_lbr:RESISTOR-0603 -> igor_lbr:RESISTOR-0805
- R10, R12, R8: value 4k7 -> 4.7k; device igor_lbr:RESISTOR-0603 -> igor_lbr:RESISTOR-0805
- R11, R13, R9: value 36 -> 22; device igor_lbr:RESISTOR-0603 -> igor_lbr:RESISTOR-0805
- R14, R15, R16, R17, R18, R19, R20, R21: value 10k -> 4.7k; device igor_lbr:RESISTOR-0603 -> igor_lbr:RESISTOR-0805
- R2: value 1k -> 4.7k; device igor_lbr:RESISTOR-0603 -> igor_lbr:RESISTOR-0805
- R4, R5: device igor_lbr:RESISTOR-0603 -> igor_lbr:RESISTOR-0805
- R6: value 220 -> 10; device igor_lbr:RESISTOR-0603 -> igor_lbr:RESISTOR-0805
- R7: value 220 -> 33; device igor_lbr:RESISTOR-0603 -> igor_lbr:RESISTOR-0805
- SW1: value B3F-3122 -> OMRON-B3W-9; device igor_lbr:SWITCH-B3F -> igor_lbr:OMRON-B3W-9
- SW10, SW11, SW12, SW13, SW14, SW15, SW16, SW17, SW18, SW19, SW2, SW20, SW21, SW22, SW3, SW4, SW5, SW6, SW7, SW8, SW9: value (none) -> OMRON-B3W-9; device igor_lbr:SWITCH-RUBBER -> igor_lbr:OMRON-B3W-9
- SW23: device igor_lbr:SWITCH-RUBBER -> igor_lbr:SWITCH-B3F
- U1, U2, U3, U4: value 4067-SO24W -> MC14067BDWR2G-SO24W; device igor_lbr:4067-SO24W -> igor_lbr:MC14067BDWR2G-SO24W
- U5: value AT90USB1286 -> STM32F405RGT6-10X10-HS; device igor_lbr:AT90USB1286 -> igor_lbr:STM32F405RGT6-10X10-HS
- U6: value 74HCT165 -> 74HC165; device igor_lbr:74HCT165 -> igor_lbr:74HC165
- U7: value 74HCT238SO -> 74238-SO; device igor_lbr:74HCT238SO -> igor_lbr:74HC238-SO
- U8: value ULN2803ADW -> ULN2803A-SO; device igor_lbr:ULN2803ADW -> igor_lbr:ULN2803A-SO
- U9: value 74HCT138SO -> 74138-SO; device igor_lbr:74HCT138SO -> igor_lbr:74HC138-SO
- VR2: value MCP1825 -> AP7343-SOT25; device igor_lbr:MCP1825 -> igor_lbr:AP7343-SOT25
- Y1: device igor_lbr:CRYSTAL -> igor_lbr:CRYSTAL-HC49
Connections:
- removed net AREF: C19.1, CONN7.1, VR2.VOUT
- removed net AREF_SELECT: C11.1, C12.1, C4.1, C5.1, CONN7.2, U1.VCC, U2.VCC, U3.VCC, U4.VCC, U5.AREF
- removed net BTLDR_EN: R3.2, SW1.1, U5.PE2(ALE/!HWB)
- removed net IN_COLUMN_0: ENC1G$1.C, ENC3G$1.C, ENC5G$1.C, ENC7G$1.C, U9.!Y0
- removed net IN_COLUMN_1: ENC2G$1.C, ENC4G$1.C, ENC6G$1.C, ENC9G$1.C, U9.!Y1
- removed net IN_COLUMN_2: ENC10G$1.C, ENC8G$1.C, U9.!Y2
- removed net IN_COLUMN_3: SW10.1, SW14.1, SW17.1, SW19.1, SW21.1, SW22.1, SW4.1, SW8.1, U9.!Y3
- removed net IN_COLUMN_4: SW12.1, SW15.1, SW16.1, SW18.1, SW2.1, SW20.1, SW23.1, SW6.1, U9.!Y4
- removed net IN_COLUMN_5: ENC1-SWITCH.1, SW13.1, SW5.1, SW9.1, U9.!Y5
- removed net IN_COLUMN_6: ENC3-SWITCH.1, SW11.1, SW3.1, SW7.1, U9.!Y6
- removed net IN_COLUMN_7: U9.!Y7
- removed net IN_ROW_0: D11.3, D12.3, D13.3, D26.3, R17.1, U6.D0
- removed net IN_ROW_1: D10.3, D2.3, D25.3, D8.3, R16.1, U6.D1
- removed net IN_ROW_2: D24.3, D4.3, D5.3, D6.3, R15.1, U6.D2
- removed net IN_ROW_3: D1.3, D23.3, D3.3, D9.3, R14.1, U6.D3
- removed net IN_ROW_4: D16.3, D21.3, R18.1, U6.D4
- removed net IN_ROW_5: D18.3, D19.3, R19.1, U6.D5
- removed net IN_ROW_6: D17.3, D20.3, R20.1, U6.D6
- removed net IN_ROW_7: D15.3, D22.3, R21.1, U6.D7
- removed net LR_1_L: D27.A, D30.A, D33.A, D36.A, D39.A, D42.A, D45.A, D48.A, R9.2
- removed net LR_1_Q: Q1.G1, R8.2, U5.PB5(PCINT5/OC.1A)
- removed net LR_2_L: D28.A, D31.A, D34.A, D37.A, D40.A, D43.A, D46.A, R11.2
- removed net LR_2_Q: Q1.G2, R10.2, U5.PB6(PCINT6/OC.1B)
- removed net LR_3_L: D29.A, D32.A, D35.A, D38.A, D41.A, D44.A, D47.A, R13.2
- removed net LR_3_Q: Q2.G2, R12.2, U5.PB4(PCINT4/OC.2A)
- removed net MISO: CONN3.1, U5.PB3(PDO/PCINT3/MISO)
- removed net MUX_COMMON_0/TDI: CONN6.9, U1.Z, U5.PF7(ADC7/TDI)
- removed net MUX_COMMON_1/TMS: CONN6.5, U2.Z, U5.PF5(ADC5/TMS)
- removed net MUX_COMMON_2/TDO: CONN6.3, U3.Z, U5.PF6(ADC6/TDO)
- removed net MUX_COMMON_3/TCK: CONN6.1, U4.Z, U5.PF4(ADC4/TCK)
- removed net N$32: D5.2, SW9.2
- removed net N$33: D5.1, SW7.2
- removed net N$34: D9.2, SW13.2
- removed net N$35: D9.1, SW11.2
- removed net N$36: D12.2, ENC1-SWITCH.2
- removed net N$40: D12.1, ENC3-SWITCH.2
- removed net RESET: CONN3.5, CONN6.6, R1.2, U5.!RESET
- removed net SDA: U5.PD1(OC2B/SDA/INT1)
- removed net SR_CLOCK: U5.PD6(T1), U6.CP
- removed net SR_LATCH: U5.PD7(T0), U6.!PL
- removed net SR_OUT: U5.PD5(XCK1), U6.Q7
- removed net TX: R6.2, U5.PD3(TXD1/INT3)
- removed net UCAP: C3.2, U5.UCAP
- removed net XTAL1: C6.1, U5.XTAL1, Y1.1
- removed net XTAL2: C7.1, U5.XTAL2, Y1.2
- new net +3V3: C10.1, C11.1, C12.1, C13.1, C15.1, C16.1, C19.1, C20.2, C21.2, C22.2, C23.1, C24.1, C4.1, C5.1, C7.1, C8.1, R14.2, R15.2, R16.2, R17.2, R18.2, R19.2, R20.2, R21.2, R7.2, U1.VCC, U2.VCC, U3.VCC, U4.VCC, U5.VBAT, U5.VDD, U5.VDD@1, U5.VDD@2, U5.VDD@4, U5.VDDA, U6.VCC, U7.E3, U7.VCC, U8.COM, U9.E3, U9.VCC, VR2.VOUT
- new net BC1: ENC1-ENC.C, ENC1-SW.1, ENC2-ENC.C, ENC2-SW.1, SW1-SW.1, U9.!Y0
- new net BC2: ENC3-ENC.C, ENC7-ENC.C, SW16-SW.1, SW3-SW.1, SW9-SW.1, U9.!Y1
- new net BC3: ENC4-ENC.C, ENC8-ENC.C, SW10-SW.1, SW17-SW.1, SW2-SW.1, U9.!Y2
- new net BC4: ENC5-ENC.C, ENC9-ENC.C, SW11-SW.1, SW18-SW.1, SW4-SW.1, U9.!Y3
- new net BC5: ENC10-ENC.C, ENC6-ENC.C, SW12-SW.1, SW19-SW.1, SW5-SW.1, U9.!Y4
- new net BC6: SW13-SW.1, SW20-SW.1, SW6-SW.1, U9.!Y5
- new net BC7: SW14-SW.1, SW21-SW.1, SW7-SW.1, U9.!Y6
- new net BC8: SW15-SW.1, SW22-SW.1, SW8-SW.1, U9.!Y7
- new net BOOT0: R1.1, U5.BOOT0
- new net BR1: D1.3, D2.3, D3.3, D4.3, R14.1, U6.D0
- new net BR2: D5.3, D6.3, D7.3, D8.3, R15.1, U6.D1
- new net BR3: D10.3, D11.3, D12.3, D9.3, R16.1, U6.D2
- new net BR4: R17.1, U6.D3
- new net BR5: D13.3, D15.3, D16.3, R18.1, U6.D4
- new net BR6: D17.3, D18.3, D19.3, R19.1, U6.D5
- new net BR7: D20.3, D21.3, D22.3, R20.1, U6.D6
- new net BR8: D23.3, D24.3, D25.3, R21.1, U6.D7
- new net BTLDR_BUTTON: R2.1, SW23.1, U5.PC4
- new net LR_1_MI: Q1.G1, R8.2, U5.PB5
- new net LR_1_MO: R9.2, SW1-LED.A, SW2-LED.A, SW3-LED.A, SW4-LED.A, SW5-LED.A, SW6-LED.A, SW7-LED.A, SW8-LED.A
- new net LR_2_MI: Q1.G2, R10.2, U5.PB4
- new net LR_2_MO: R11.2, SW10-LED.A, SW11-LED.A, SW12-LED.A, SW13-LED.A, SW14-LED.A, SW15-LED.A, SW9-LED.A
- new net LR_3_MI: Q2.G2, R12.2, U5.PB3
- new net LR_3_MO: R13.2, SW16-LED.A, SW17-LED.A, SW18-LED.A, SW19-LED.A, SW20-LED.A, SW21-LED.A, SW22-LED.A
- new net MIDI_OUT: R6.2, U5.PB10
- new net MUX_COMMON_1: U1.Z, U5.PA3
- new net MUX_COMMON_2: U2.Z, U5.PA0
- new net MUX_COMMON_3: U3.Z, U5.PA1
- new net MUX_COMMON_4: U4.Z, U5.PA2
- new net N$10: D3.2, SW5-SW.2
- new net N$11: D3.1, SW6-SW.2
- new net N$13: C6.1, U5.VCAP@2
- new net N$5: D1.1, SW1-SW.2
- new net N$8: D2.1, SW4-SW.2
- new net N$9: D1.2, SW3-SW.2
- new net NRST: C27.1, U5.NRST
- new net OSC_IN: C25.1, U5.PH0, Y1.1
- new net OSC_OUT: C26.1, U5.PH1, Y1.2
- new net SR_IN_CLOCK: U5.PC15, U6.CP
- new net SR_IN_DATA: U5.PC14, U6.Q7
- new net SR_IN_LATCH: U5.PC13, U6.!PL
- new net SWDCLK: CONN3.1, U5.PA14
- new net SWDIO: CONN3.2, U5.PA13
- new net USB_SHIELD: CONN1-S1.S, CONN1-S2.S, L1.1
- net +5V: now also CONN1-USB.VBUS, R2.2, VR2.EN; no longer C10.1, C13.1, C15.1, C16.1, C20.2, C21.2, C22.2, C23.1, C24.1, C8.1, CONN1G$1.VBUS, CONN3.2, CONN6.4, CONN7.3, R1.1, R14.2, R15.2, R16.2, R17.2, R18.2, R19.2, R2.1, R20.2, R21.2, R3.1, R7.2, U5.AVCC, U5.UVCC, U5.VBUS, U5.VCC, U5.VCC@1, U6.VCC, U7.E3, U7.VCC, U8.COM, U9.E3, U9.VCC
- net D+: now also U5.PA12; no longer U5.D+
- net D+X: now also CONN1-USB.D+; no longer CONN1G$1.D+
- net D-: now also U5.PA11; no longer U5.D-
- net D-X: now also CONN1-USB.D-; no longer CONN1G$1.D-
- net DEC_IN_A0: now also U5.PC8; no longer U5.PC3(A11/T.3)
- net DEC_IN_A1: now also U5.PC7; no longer U5.PC4(A12/OC.3C)
- net DEC_IN_A2: now also U5.PC6; no longer U5.PC5(A13/OC.3A)
- net DEC_OUT_A0: now also U5.PB9; no longer U5.PC0(A8)
- net DEC_OUT_A1: now also U5.PB7; no longer U5.PC1(A9)
- net DEC_OUT_A2: now also U5.PB6; no longer U5.PC2(A10)
- net E10_A: now also D22.1, ENC10-ENC.A; no longer D25.1, ENC10G$1.A
- net E10_B: now also D25.1, ENC10-ENC.B; no longer D26.1, ENC10G$1.B
- net E1_A: now also D13.1, ENC1-ENC.A; no longer D3.1, ENC1G$1.A
- net E1_B: now also D17.1, ENC1-ENC.B; no longer D6.1, ENC1G$1.B
- net E2_A: now also D20.1, ENC2-ENC.A; no longer D10.1, ENC3G$1.A
- net E2_B: now also D23.1, ENC2-ENC.B; no longer D13.1, ENC3G$1.B
- net E3_A: now also D13.2, ENC3-ENC.A; no longer D16.1, ENC5G$1.A
- net E3_B: now also D17.2, ENC3-ENC.B; no longer D18.1, ENC5G$1.B
- net E4_A: now also D15.1, ENC4-ENC.A; no longer D20.1, ENC7G$1.A
- net E4_B: now also D18.1, ENC4-ENC.B; no longer D22.1, ENC7G$1.B
- net E5_A: now also D15.2, ENC5-ENC.A; no longer D3.2, ENC9G$1.A
- net E5_B: now also D18.2, ENC5-ENC.B; no longer D6.2, ENC9G$1.B
- net E6_A: now also D16.1, ENC6-ENC.A; no longer D10.2, ENC2G$1.A
- net E6_B: now also D19.1, ENC6-ENC.B; no longer D13.2, ENC2G$1.B
- net E7_A: now also D20.2, ENC7-ENC.A; no longer D16.2, ENC4G$1.A
- net E7_B: now also D23.2, ENC7-ENC.B; no longer D18.2, ENC4G$1.B
- net E8_A: now also D21.1, ENC8-ENC.A; no longer D20.2, ENC6G$1.A
- net E8_B: now also D24.1, ENC8-ENC.B; no longer D22.2, ENC6G$1.B
- net E9_A: now also D21.2, ENC9-ENC.A; no longer D23.1, ENC8G$1.A
- net E9_B: now also D24.2, ENC9-ENC.B; no longer D24.1, ENC8G$1.B
- net GND: now also C25.2, C26.2, C27.2, CONN1-USB.GND, CONN3.3, ENC1-S1.S, ENC1-S2.S, ENC10-S1.S, ENC10-S2.S, ENC2-S1.S, ENC2-S2.S, ENC3-S1.S, ENC3-S2.S, ENC4-S1.S, ENC4-S2.S, ENC5-S1.S, ENC5-S2.S, ENC6-S1.S, ENC6-S2.S, ENC7-S1.S, ENC7-S2.S, ENC8-S1.S, ENC8-S2.S, ENC9-S1.S, ENC9-S2.S, R1.2, SW23.2, U5.VSS, U5.VSS@1, U5.VSSA; no longer CONN1G$1.GND, CONN3.6, CONN6.10, CONN6.2, D7.C, ENC10G$2.S, ENC10G$3.S, ENC1G$2.S, ENC1G$3.S, ENC2G$2.S, ENC2G$3.S, ENC3G$2.S, ENC3G$3.S, ENC4G$2.S, ENC4G$3.S, ENC5G$2.S, ENC5G$3.S, ENC6G$2.S, ENC6G$3.S, ENC7G$2.S, ENC7G$3.S, ENC8G$2.S, ENC8G$3.S, ENC9G$2.S, ENC9G$3.S, SW1.2, U5.GND, U5.GND@1, U5.GND@2, U5.UGND, VR2.GND@1
- net LCD_CS: now also U5.PC11; no longer U5.PA4(AD4)
- net LCD_DC: now also U5.PD2; no longer U5.PA3(AD3)
- net LCD_RESET: now also U5.PA15; no longer U5.PA5(AD5)
- net LC_1: now also SW15-LED.C, SW22-LED.C, SW8-LED.C; no longer D27.C, D28.C, D29.C
- net LC_2: now also SW14-LED.C, SW21-LED.C, SW7-LED.C; no longer D30.C, D31.C, D32.C
- net LC_3: now also SW13-LED.C, SW20-LED.C, SW6-LED.C; no longer D33.C, D34.C, D35.C
- net LC_4: now also SW12-LED.C, SW19-LED.C, SW5-LED.C; no longer D36.C, D37.C, D38.C
- net LC_5: now also SW11-LED.C, SW18-LED.C, SW4-LED.C; no longer D39.C, D40.C, D41.C
- net LC_6: now also SW10-LED.C, SW17-LED.C, SW3-LED.C; no longer D42.C, D43.C, D44.C
- net LC_7: now also SW16-LED.C, SW2-LED.C, SW9-LED.C; no longer D45.C, D46.C, D47.C
- net LC_8: now also SW1-LED.C; no longer D48.C
- net MOSI: now also U5.PC12; no longer CONN3.4, U5.PB2(PDI/PCINT2/MOSI)
- net MUX_S0: now also U5.PB12; no longer U5.PF1(ADC1)
- net MUX_S1: now also U5.PB13; no longer U5.PF0(ADC0)
- net MUX_S2: now also U5.PB15; no longer U5.PF2(ADC2)
- net MUX_S3: now also U5.PB14; no longer U5.PF3(ADC3)
- net N$12: now also C3.2, U5.VCAP; no longer CONN1G$2.S, CONN1G$3.S, L1.1
- net N$14: now also D4.2, SW7-SW.2; no longer D1.2, SW4.2
- net N$15: now also D4.1, SW8-SW.2; no longer D1.1, SW2.2
- net N$16: now also D5.2, ENC1-SW.2; no longer D4.2, SW8.2
- net N$17: now also D6.2, SW10-SW.2; no longer D4.1, SW6.2
- net N$18: now also D6.1, SW11-SW.2; no longer D8.1, SW10.2
- net N$19: now also D7.1, SW12-SW.2; no longer D8.2, SW12.2
- net N$20: now also D7.2, SW13-SW.2; no longer D11.1, SW14.2
- net N$21: now also D8.2, SW14-SW.2; no longer D11.2, SW15.2
- net N$22: now also D8.1, SW15-SW.2; no longer D15.2, SW17.2
- net N$23: now also D5.1, SW9-SW.2; no longer D15.1, SW16.2
- net N$24: now also D9.2, ENC2-SW.2; no longer D17.2, SW19.2
- net N$25: now also D9.1, SW16-SW.2; no longer D17.1, SW18.2
- net N$26: now also D10.2, SW17-SW.2; no longer D19.2, SW21.2
- net N$27: now also D10.1, SW18-SW.2; no longer D19.1, SW20.2
- net N$28: now also D11.2, SW19-SW.2; no longer D21.1, SW22.2
- net N$29: now also D11.1, SW20-SW.2; no longer D21.2, SW23.2
- net N$30: now also D12.2, SW21-SW.2; no longer D2.2, SW5.2
- net N$31: now also D12.1, SW22-SW.2; no longer D2.1, SW3.2
- net N$6: now also D2.2, SW2-SW.2; no longer D7.A, R2.2
- net SCLK: now also U5.PC10; no longer CONN3.3, U5.PB1(PCINT1/SCLK)
Other:
- note added: "IN MATRIX"
- note added: "LED MATRIX"
- note added: "VBAT"
- note added: "VDD1"
- note added: "VDD2"
- note added: "VDD3"
- note added: "VDD4"
- note added: "VDDA"
- note removed: "ANALOG"
- note removed: "AVCC/64"
- note removed: "ENCODERS/BUTTONS"
- note removed: "ICSP"
- note removed: "JTAG"
- note removed: "UVCC/3"
- note removed: "VBUS/8"
- note removed: "VCC/21"
- note removed: "VCC/52"
- moved on the sheet: C1, CONN2, CONN4, CONN5, D10, D11, D12, D13, D14, D15, D16, D17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
